Commit message: render mode added + ZMP bug fix + urdf update

File: bullet_sim/surena4.urdf (robot description, URDF)
Before this commit: robot rrbot, 29 links, 28 joints
Links:
- link LARM_LINK3: geometry collision mesh filename=package://bullet_sim/meshes/Upper-arm-Left.STL; visual mesh filename=package://bullet_sim/meshes/Upper-arm-Left.STL
- link LARM_LINK4: geometry visual mesh filename=package://bullet_sim/meshes/fore-arm-Left.STL
- link LARM_LINK7: geometry collision mesh filename=package://bullet_sim/meshes/Hand-Left.STL; visual mesh filename=package://bullet_sim/meshes/Hand-Left.STL
- link LLeg_Foot_Link: geometry collision box size=0.26 0.16 0.02; visual mesh filename=package://bullet_sim/meshes/Foot-Left.STL
- link LLeg_Hip_Shank_Link: geometry collision cylinder length=0.35 radius=0.04; visual mesh filename=package://bullet_sim/meshes/Shank-Left.STL
- link LLeg_Hip_Thigh_Link: geometry collision cylinder length=0.35 radius=0.04; visual mesh filename=package://bullet_sim/meshes/Thigh-Left.STL
- link RARM_LINK3: geometry collision mesh filename=package://bullet_sim/meshes/Upper-arm-right.STL; visual mesh filename=package://bullet_sim/meshes/Upper-arm-right.STL
- link RARM_LINK4: geometry visual mesh filename=package://bullet_sim/meshes/fore-arm-right.STL
- link RARM_LINK7: geometry collision mesh filename=package://bullet_sim/meshes/Hand-Right.STL; visual mesh filename=package://bullet_sim/meshes/Hand-Right.STL
- link RLeg_Foot_Link: geometry collision box size=0.26 0.16 0.02; visual mesh filename=package://bullet_sim/meshes/Foot-Right.STL
- link RLeg_Hip_Shank_Link: geometry collision cylinder length=0.35 radius=0.04; visual mesh filename=package://bullet_sim/meshes/Shank-Right.STL
- link RLeg_Hip_Thigh_Link: geometry collision cylinder length=0.35 radius=0.04; visual mesh filename=package://bullet_sim/meshes/Thigh-Right.STL
- link WAIST_LINK2: geometry collision mesh filename=package://bullet_sim/meshes/tORSO.STL; visual mesh filename=package://bullet_sim/meshes/tORSO.STL
- link pelvis: geometry collision cylinder length=0.23 radius=0.08; visual mesh filename=package://bullet_sim/meshes/pelvis.STL
